Commit message: Controller implemented but not deployed or tested

File: catkin_ws/src/human_arm_description/urdf/human_arm_description.urdf (robot description, URDF)
Before this commit: robot human_arm, 11 links, 10 joints
Links:
- removed link world
- link Scaphant: mass 0.0290597320457 -> 8.21933343559e-06; geometry visual cylinder length=0.00141421356237 radius=0.001
- link base_link: mass 0.581194640914 -> 8.21933343559e-06; geometry visual cylinder length=0.00141421356237 radius=0.001
Joints:
- removed joint joint_world_base_link
- joint joint_Scaphant_Humphant: origin xyz=0.05 -0.0 0.0 rpy=0.0 -0.0 0.0 -> xyz=0.001 -0.0 0.001 rpy=0.0 -0.0 0.0
- joint joint_base_link_Scaphant: origin xyz=0.0 -0.0 1.0 rpy=0.0 -0.0 1.57079632679 -> xyz=0.001 -0.0 0.001 rpy=0.0 -0.0 1.57079632679

File: catkin_ws/src/human_arm_description/urdf/human_arm_description.urdf.xacro (robot description, xacro)
@@ -147,8 +147,8 @@
     alpha="${radians(-90)}"/>
     <xacro:frame_pair parent="Hand"/>
-  <gazebo>
+  <!--<gazebo>
     <plugin name="gazebo_ros_control" filename="libgazebo_ros_control.so">
       <robotNamespace>/</robotNamespace>
     </plugin>
-  </gazebo>
+  </gazebo>-->
 </robot>

Commit message: Fix collide

File: catkin_ws/src/human_arm_description/urdf/human_arm_description.urdf (robot description, URDF)
Before this commit: robot human_arm, 10 links, 9 joints
Links:
- link Hand: mass None -> 4.64955712731; geometry collision cylinder length=0.08 radius=0.01; visual cylinder length=0.08 radius=0.01
- link Humerus: mass 0.00570933146923 -> 16.8778923721; geometry collision cylinder length=0.2904 radius=0.01; visual cylinder length=0.2904 radius=0.01
- link Humphant: mass 8.21933343559e-06 -> 0.145298660229; geometry collision cylinder length=0.01 radius=0.005; visual cylinder length=0.01 radius=0.005
- link Humphant1: mass 0.168778923721 -> 0.145298660229; geometry collision cylinder length=0.01 radius=0.005; visual cylinder length=0.01 radius=0.005
- link Lunate: mass 8.21933343559e-06 -> 0.145298660229; geometry collision cylinder length=0.01 radius=0.005; visual cylinder length=0.01 radius=0.005
- link Radius: mass 0.0180347422283 -> 14.9657620035; geometry collision cylinder length=0.2575 radius=0.01; visual cylinder length=0.2575 radius=0.01
- link Scaphant: mass 8.21933343559e-06 -> 0.145298660229; geometry collision cylinder length=0.01 radius=0.005; visual cylinder length=0.01 radius=0.005
- link Ulna: mass 0.149657620035 -> 0.570933146923; geometry collision cylinder length=0.00982344135219 radius=0.01; visual cylinder length=0.00982344135219 radius=0.01
- link Z6: mass 8.21933343559e-06 -> 1.80347422283; geometry collision cylinder length=0.0310304688975 radius=0.01; visual cylinder length=0.0310304688975 radius=0.01
- link base_link: mass 8.21933343559e-06 -> 0.145298660229; geometry collision cylinder length=0.01 radius=0.005; visual cylinder length=0.01 radius=0.005
Joints:
- joint joint_Humerus_Ulna: limit lower=0 upper=6.28318530718 effort=1000.0 velocity=0.5 -> lower=0.0 upper=2.26892802759 effort=1000.0 velocity=0.5
- joint joint_Humphant1_Humerus: limit lower=0 upper=6.28318530718 effort=1000.0 velocity=0.5 -> lower=-3.83972435439 upper=1.91986217719 effort=1000.0 velocity=0.5
- joint joint_Humphant_Humphant1: limit lower=0 upper=6.28318530718 effort=1000.0 velocity=0.5 -> lower=0.0 upper=3.14159265359 effort=1000.0 velocity=0.5; origin xyz=0.001 -0.001 6.12323399574e-20 rpy=1.57079632679 -0.0 0.0 -> xyz=0.0 -0.0 0.0 rpy=1.57079632679 -0.0 0.0
- joint joint_Lunate_Hand: origin xyz=0.001 0.001 6.12323399574e-20 rpy=-0.785398163397 -1.57079632679 -0.785398163397 -> xyz=-0.08 0.0 0.0 rpy=-0.785398163397 -1.57079632679 -0.785398163397
- joint joint_Radius_Z6: limit lower=0 upper=6.28318530718 effort=1000.0 velocity=0.5 -> lower=-0.174532925199 upper=0.436332312999 effort=1000.0 velocity=0.5; origin xyz=0.0105 0.0289298369418 0.00396289471508 rpy=-2.18090776315 -1.33165554748 -2.54497002525 -> xyz=-0.0105 0.0289298369418 0.00396289471508 rpy=-2.18090776315 -1.33165554748 -2.54497002525
- joint joint_Scaphant_Humphant: limit lower=0 upper=6.28318530718 effort=1000.0 velocity=0.5 -> lower=-1.57079632679 upper=2.26892802759 effort=1000.0 velocity=0.5; origin xyz=0.001 -0.0 0.001 rpy=0.0 -0.0 0.0 -> xyz=0.0 -0.0 0.0 rpy=0.0 -0.0 0.0
- joint joint_Ulna_Radius: limit lower=0 upper=6.28318530718 effort=1000.0 velocity=0.5 -> lower=-1.57079632679 upper=1.57079632679 effort=1000.0 velocity=0.5
- joint joint_Z6_Lunate: limit lower=0 upper=6.28318530718 effort=1000.0 velocity=0.5 -> lower=-0.610865238198 upper=0.610865238198 effort=1000.0 velocity=0.5; origin xyz=0.001 0.000573576436351 -0.000819152044289 rpy=-2.54422044057 0.13626609681 -0.197095295237 -> xyz=0.0 0.0 -0.0 rpy=-2.54422044057 0.13626609681 -0.197095295237
- joint joint_base_link_Scaphant: origin xyz=0.001 -0.0 0.001 rpy=0.0 -0.0 1.57079632679 -> xyz=0.0 -0.0 0.0 rpy=0.0 -0.0 1.57079632679

Commit message: Further scale of weight

File: catkin_ws/src/human_arm_description/urdf/human_arm_description.urdf (robot description, URDF)
Before this commit: robot human_arm, 10 links, 9 joints
Links:
- link Hand: mass 4.64955712731 -> 464.955712731
- link Humerus: mass 16.8778923721 -> 1687.78923721
- link Humphant: mass 0.145298660229 -> 14.5298660229
- link Humphant1: mass 0.145298660229 -> 14.5298660229
- link Lunate: mass 0.145298660229 -> 14.5298660229
- link Radius: mass 14.9657620035 -> 1496.57620035
- link Scaphant: mass 0.145298660229 -> 14.5298660229
- link Ulna: mass 0.570933146923 -> 57.0933146923
- link Z6: mass 1.80347422283 -> 180.347422283
- link base_link: mass 0.145298660229 -> 14.5298660229

File: catkin_ws/src/human_arm_description/urdf/human_arm_description.xacro (robot description, xacro)
@@ -2,5 +2,5 @@
 <robot xmlns:xacro="http://www.ros.org/wiki/xacro" name="human_arm">
     <xacro:property name="scale" value="${1}" />
-    <xacro:property name="bone_density" value="${1850 * 100}" />
+    <xacro:property name="bone_density" value="${1850 * 10000}" />
     <xacro:property name="len_humerus_y" value="${0.2904*scale}" />
     <xacro:property name="len_ulna_z" value="${0.0200*scale}" />
